File: Y-pcbv1/solarpcd.kicad_pcb (KiCad board)
At the start: 6 copper layers, 239.3 x 99.4 mm, 66 parts, among them IC2 TSL2561, J1 XF2M-1015-1A, U1 SWLP.12.B, U2 Value, U3 TSL2561, U3 kill_switch, U4 kill_switch, X1 mainboard-rescue_ANTENNA_U.FL-

Commit message: killer coils
Parts:
- removed D3: MSS1P4-M3_89A, custom-footprints:MICROSMP
- removed X1: mainboard-rescue_ANTENNA_U.FL-, Connector_Coaxial:U.FL_Hirose_U.FL-R-SMT-1_Vertical
- added D30: MSS1P4-M3_89A, custom-footprints:MICROSMP, B.Cu at (159.4, 87.2)
- added J2: U.FL-R-SMT-1, custom-footprints:U.FL-R-SMT-1, B.Cu at (153.9, 108.8)
- D1: value SDM20U40-7 -> BZT52C4V7t
- moved IC2 26.1 mm to (104.2, 86.0)
- moved R10 26.1 mm to (103.5, 83.6)
- moved R9 26.1 mm to (104.5, 83.6)
- moved R19 7.77 mm to (100.5, 90.4)
- moved R3 7.77 mm to (100.5, 91.8)
- moved R2 7.77 mm to (99.5, 91.8)
- moved R4 7.77 mm to (99.5, 90.4)
- renumbered C14 to C13, C13 to C14, U3 to IC2, R13 to R10, R14 to R11, R15 to R12, R16 to R13, R17 to R14, R18 to R15, R5 to R2, R6 to R3, R7 to R4, R8 to R5, R9 to R6, R10 to R7, R11 to R8, R12 to R9
Connections:
- C10 pad 1: Net-(C10-Pad1) -> +3V3
- C12 pad 1: Net-(C10-Pad1) -> +3V3
- C7 pad 1: Net-(C10-Pad1) -> +3V3
- D11 pad 1: VSOLAR -> Net-(D11-Pad1)
- IC2 pad 2: Net-(R12-Pad1) -> Net-(IC2-Pad2)
- IC2 pad 5: Net-(U3-Pad5) -> Net-(IC2-Pad5)
- IC2 pad 5: (no net) -> Net-(IC2-Pad5)
- L2 pad 2: Net-(C10-Pad1) -> +3V3
- R10 pad 2: Net-(R12-Pad1) -> Net-(IC2-Pad2)
- R9 pad 1: Net-(R12-Pad1) -> Net-(IC2-Pad2)
- SC1 pad 1: VSOLAR -> Net-(D11-Pad1)
- SC3 pad 1: VSOLAR -> Net-(D11-Pad1)
- SC5 pad 1: VSOLAR -> Net-(D11-Pad1)
- U2 pad 14: Net-(C10-Pad1) -> +3V3
Routing:
- net Net-(D11-Pad1): track 0.00 -> 36.6 mm, vias 0 -> 2
- net VSOLAR: track 39.9 -> 6.82 mm
- net Net-(R2-Pad2): track 7.04 -> 0.00 mm, vias 2 -> 0
- net Net-(R10-Pad2): track 0.00 -> 7.04 mm, vias 0 -> 2
- net Net-(C10-Pad1): track 9.20 -> 7.73 mm
- net +3V3: track 11.6 -> 13.0 mm
- net Net-(D3-Pad2): track 1.42 -> 0.00 mm, vias 2 -> 0
- added copper zone on B.Cu, net +3V3
- removed copper zone on B.Cu, net Net-(C10-Pad1)

Commit message: -Y board finished
Parts:
- removed D4, D5: SBDiode, SolarCellParts:SB Diode
- removed the IC2 at (340.4, 129.5)
- removed REF**: Gauge_10mm_Type1_SilkScreenTop, Calibration_Scale:Gauge_10mm_Type1_SilkScreenTop
- removed Ref**: Val**, custom-footprints:xpanel
- removed the SC1 at (313.1, 164.8)
- removed the SC2 at (305.6, 155.5)
- removed the SC3 at (305.6, 146.3)
- removed the SC4 at (305.6, 137.3)
- removed the SC5 at (312.9, 125.8)
- removed the SC6 at (329.6, 137.3)
- removed SC7, SC8: SolarCell_Small, SolarCellParts:KXOB25-05X3F
- added J3: BATTERY CONNECTOR, custom-footprints:SCREWTERMINAL-3.5MM-2_LOCK, B.Cu at (130.4, 100.1)
- U3: value kill_switch -> SW_SPDT; footprint solarpcb:D2F-L2 -> custom-footprints:D2F-L2
- U4: value kill_switch -> SW_SPDT; footprint solarpcb:D2F-L2-2 -> custom-footprints:D2F-L2
- moved C5 194.4 mm to (143.9, 114.4), turned to 180 degrees
- moved IC2 50.0 mm to (143.8, 116.6)
- moved R10 49.9 mm to (140.5, 117.1), turned to 90 degrees
- moved R9 48.5 mm to (140.5, 116.1), turned to 90 degrees
- moved R19 45.2 mm to (145.4, 85.3)
- moved R3 45.2 mm to (145.4, 86.7)
- moved R4 45.2 mm to (144.4, 85.3)
- moved R2 45.2 mm to (144.4, 86.7)
- moved U4 0.13 mm to (130.4, 107.4)
Connections:
- D2 pad 2: Net-(C10-Pad1) -> +3V3
- U3 pad 1: (no net) -> Net-(U3-Pad1)
- U3 pad 2: BATT_P -> Net-(J3-Pad2)
- U3 pad 3: (no net) -> BATT_P
- U4 pad 1: (no net) -> Net-(U4-Pad1)
- U4 pad 2: BATT_N -> Net-(J3-Pad1)
- U4 pad 3: (no net) -> BATT_N
Routing:
- net /coil: track 3.61 -> 16503.7 mm, vias 2 -> 7
- net COIL_N: track 16448.2 -> 31.4 mm, vias 5 -> 2
- net BATT_N: track 1.71 -> 55.6 mm, vias 0 -> 1
- net BATT_P: track 2.87 -> 55.7 mm, vias 0 -> 1
- net GND: track 150.2 -> 189.9 mm, vias 8 -> 19
- net +3V3: track 13.0 -> 46.0 mm
- net SCL1: track 1.15 -> 31.8 mm, vias 1 -> 2
- net COIL_P: track 0.00 -> 30.1 mm, vias 0 -> 2
- net SDA1: track 2.04 -> 29.7 mm, vias 1 -> 2
- net Net-(C10-Pad1): track 7.73 -> 0.00 mm
- net Net-(R2-Pad2): track 0.00 -> 7.46 mm, vias 0 -> 2
- net Net-(J3-Pad1): track 0.00 -> 7.11 mm
- net Net-(R10-Pad2): track 7.04 -> 0.00 mm, vias 2 -> 0
- net Net-(J3-Pad2): track 0.00 -> 5.85 mm
- net Net-(IC2-Pad2): track 0.00 -> 1.80 mm
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Other:
- board size 239.3 x 99.4 mm -> 64 x 58 mm
- board text removed: "3V3"
- board text removed: "GND"
- board text removed: "sig"

Commit message: zipped fabrication files for all but +Y
Parts:
- added Ref**: Val**, custom-footprints:ypanel, B.Cu at (161.9, 85.6)
- added Ref**: Val**, custom-footprints:ypanel, F.Cu at (169.6, 85.9)
Other:
- board text removed: "Coil +"
- board text removed: "Coil -"
