File: Y-pcbv1/solarpcd.sch (KiCad schematic (older format))
At the start: 48 parts, among them IC2 TSL2561, J1 XF2M-1015-1A, U1 SWLP.12.B, U2 Value, U3 kill_switch, U4 kill_switch, X1 mainboard-rescue_ANTENNA_U.FL-

Commit message: killer coils
Parts:
- removed D?: D_Schottky, custom-footprints:MICROSMP, symbol Device:D_Schottky
- removed X1: mainboard-rescue_ANTENNA_U.FL-, Connector_Coaxial:U.FL_Hirose_U.FL-R-SMT-1_Vertical, symbol solarpcd-rescue:mainboard-rescue_ANTENNA_U.FL--mainboard-cache
- added D30: MSS1P4-M3_89A, MICROSMP, symbol symbols:MSS1P4-M3_89A
- added J2: U.FL-R-SMT-1, custom-footprints:U.FL-R-SMT-1, symbol symbols:U.FL-R-SMT-1
- added R16: 0, Resistor_SMD:R_0402_1005Metric, symbol solarpcd-rescue:0OHM-0603-1_10W-5%-misc-circuits-cache-misc-circuits-rescue
Connections:
- net labels added: coil
- wire segments 178 -> 169
Other:
- moved on the sheet: J1, U1

Commit message: -Y board finished
Parts:
- removed C1: 1.0uF, Capacitor_SMD:C_0402_1005Metric, symbol solarpcd-rescue:1.0UF-0603-16V-10%-misc-circuits-cache-misc-circuits-rescue
- removed C10, C14, C2, C9: 0.1uF, Capacitor_SMD:C_0402_1005Metric, symbol solarpcd-rescue:0.1UF-0603-25V-(+80_-20%)-misc-circuits-cache-misc-circuits-res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
- removed C11, C12, C13, C6: 100uF, Capacitor_SMD:C_0603_1608Metric, symbol solarpcd-rescue:0.1UF-0603-25V-(+80_-20%)-misc-circuits-cache-misc-circuits-res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
- removed C3, C8: 4.7uF, Capacitor_SMD:C_0402_1005Metric, symbol solarpcd-rescue:4.7UF0603-misc-circuits-cache-misc-circuits-rescue
- removed C4: 10nF, Capacitor_SMD:C_0402_1005Metric, symbol solarpcd-rescue:10NF-0603-50V-10%-misc-circuits-cache-misc-circuits-rescue
- removed C7: 22uF, Capacitor_SMD:C_0402_1005Metric, symbol solarpcd-rescue:22UF-0805-6.3V-20%-misc-circuits-cache-misc-circuits-rescue
- removed D1: BZT52C4V7t, solarpcb:SOD523, symbol solarpcd-rescue:DIODE-SOD523-misc-circuits-cache-misc-circuits-rescue
- removed L1: 22uH-LPS4018-223MR, solarpcb:LPS4018, symbol solarpcd-rescue:COILCRAFT-LPS4018-misc-circuits-cache-misc-circuits-rescue
- removed L2: 10uH-LPS4018-103MR, solarpcb:LPS4018, symbol solarpcd-rescue:COILCRAFT-LPS4018-misc-circuits-cache-misc-circuits-rescue
- removed R1, R11, R12, R13, R14, R15: 0, Resistor_SMD:R_0402_1005Metric, symbol solarpcd-rescue:0OHM-0603-1_10W-5%-misc-circuits-cache-misc-circuits-rescue
- removed R2: 7.32M, Resistor_SMD:R_0402_1005Metric, symbol solarpcd-rescue:1MOHM-0603-1_4W-5%-misc-circuits-cache-misc-circuits-rescue
- removed R3: 5.62M, Resistor_SMD:R_0402_1005Metric, symbol solarpcd-rescue:1MOHM-0603-1_4W-5%-misc-circuits-cache-misc-circuits-rescue
- removed R4: 374K, Resistor_SMD:R_0402_1005Metric, symbol solarpcd-rescue:1MOHM-0603-1_4W-5%-misc-circuits-cache-misc-circuits-rescue
- removed R5, R7: 8.25M, Resistor_SMD:R_0402_1005Metric, symbol solarpcd-rescue:1MOHM-0603-1_4W-5%-misc-circuits-cache-misc-circuits-rescue
- removed R6: 4.53M, Resistor_SMD:R_0402_1005Metric, symbol solarpcd-rescue:1MOHM-0603-1_4W-5%-misc-circuits-cache-misc-circuits-rescue
- removed R8: 4.75M, Resistor_SMD:R_0402_1005Metric, symbol solarpcd-rescue:1MOHM-0603-1_4W-5%-misc-circuits-cache-misc-circuits-rescue
- removed U2: Value, solarpcb:QFN50P350X350X100-21N-D, symbol solarpcd-rescue:BQ25570RGRR-misc-circuits-cache-misc-circuits-rescue
- removed U3: kill_switch, solarpcb:D2F-L2, symbol solarpcd_lib:kill_switch
- removed U4: kill_switch, solarpcb:D2F-L2-2, symbol solarpcd_lib:kill_switch
- added J3: BATTERY CONNECTOR, custom-footprints:SCREWTERMINAL-3.5MM-2_LOCK, symbol Connector:Screw_Terminal_01x02
- added U3, U4: SW_SPDT, custom-footprints:D2F-L2, symbol Switch:SW_SPDT
Connections:
- net BATT_N: now also U4.3 (C)
- net BATT_P: now also U3.3 (C)
- new net: J3.2 (Pin_2), U3.2 (B)
- new net: J3.1 (Pin_1), U4.2 (B)
Other:
- note removed: "80% MPPT"
- note removed: "BQ25570RGRR"
- note removed: "DNI"
- note removed: "Energy Harvesting IC"
- note removed: "External energy storage\nInput/Output"
- note removed: "External\nPower Source\nInput\n(Solar)"
- note removed: "Imin=280uA"
- note removed: "MPPT Set Resistors"
- note removed: "Sets of resistor dividers should = 13MOhm"
- note removed: "VBAT_OK\nON: 3.51V\nOFF: 3.42V"
- note removed: "VBAT_OV\n4.2V"
- note removed: "VOUT=1.21V*((ROUT2+ROUT1)/ROUT1)"
- note removed: "VOUT\n3.31"
- note removed: "ZENER"

Commit message: Updated -Y PCB design
Parts:
- D30: footprint MICROSMP -> solarpcb:MICROSMP; symbol symbols:MSS1P4-M3_89A -> solarpcd-rescue:MSS1P4-M3_89A-symbols
- J2: symbol symbols:U.FL-R-SMT-1 -> solarpcd-rescue:U.FL-R-SMT-1-symbols
- J3: symbol Connector:Screw_Terminal_01x02 -> solarpcd-rescue:Screw_Terminal_01x02-Connector
- U3: footprint custom-footprints:D2F-L2 -> solarpcb:D2F-L2-2; symbol Switch:SW_SPDT -> solarpcd-rescue:SW_SPDT-Switch
- U4: footprint custom-footprints:D2F-L2 -> solarpcb:D2F-L2; symbol Switch:SW_SPDT -> solarpcd-rescue:SW_SPDT-Switch
Changed lines of the file:
@@
 	8750 5000 8600 5000
 $Comp
-L power:GND #PWR0108
+L solarpcd-rescue:GND-power #PWR0108
 U 1 1 5DB779CC
 P 9150 5300
@@
 $EndComp
 $Comp
-L power:+3V3 #PWR0110
+L solarpcd-rescue:+3V3-power #PWR0110
 U 1 1 5DB87DA5
 P 8750 5200
@@
 	7650 6600 7400 6600
 $Comp
-L power:GND #PWR0111
+L solarpcd-rescue:GND-power #PWR0111
 U 1 1 5DB1FC5C
 P 5800 6900
@@
 	6100 6100 5800 6100
 $Comp
-L power:+3V3 #PWR0112
+L solarpcd-rescue:+3V3-power #PWR0112
 U 1 1 5DB2D712
 P 5800 6100
@@
 	8750 5400 8600 5400
 $Comp
-L power:GND #PWR0113
+L solarpcd-rescue:GND-power #PWR0113
 U 1 1 5DB7ADC7
 P 7200 5300
@@
 	4500 6300 4500 6400
 $Comp
-L power:GND #PWR0114
+L solarpcd-rescue:GND-power #PWR0114
 U 1 1 5DB6D916
 P 4500 6400
@@
 BATT_P
 $Comp
-L symbols:MSS1P4-M3_89A D30
+L solarpcd-rescue:MSS1P4-M3_89A-symbols D30
 U 1 1 5DB46377
 P 950 6200
 F 0 "D30" H 1250 6465 50  0000 C CNN
 F 1 "MSS1P4-M3_89A" H 1250 6374 50  0000 C CNN
-F 2 "MICROSMP" H 1350 6350 50  0001 L BNN
+F 2 "solarpcb:MICROSMP" H 1350 6350 50  0001 L BNN
 F 3 "https://www.vishay.com/docs/89019/mss1p4.pdf" H 1350 6250 50  0001 L BNN
 F 4 "Vishay MSS1P4-M3/89A SMT Schottky Diode, 40V 1A, 2-Pin uSMP" H 1350 6150 50  0001 L BNN "Description"
@@
 	8600 5300 9150 5300
 $Comp
-L symbols:U.FL-R-SMT-1 J2
+L solarpcd-rescue:U.FL-R-SMT-1-symbols J2
 U 1 1 5DC33039
 P 6950 8300
@@
 	7000 8950 7000 8900
 $Comp
-L power:GND #PWR0115
+L solarpcd-rescue:GND-power #PWR0115
 U 1 1 5DC4B261
 P 6800 9000
@@
 COIL_N
 $Comp
-L Switch:SW_SPDT U3
+L solarpcd-rescue:SW_SPDT-Switch U3
 U 1 1 5DC81E30
 P 10550 4600
 F 0 "U3" H 10550 4885 50  0000 C CNN
 F 1 "SW_SPDT" H 10550 4794 50  0000 C CNN
-F 2 "custom-footprints:D2F-L2" H 10550 4600 50  0001 C CNN
+F 2 "solarpcb:D2F-L2-2" H 10550 4600 50  0001 C CNN
 F 3 "~" H 10550 4600 50  0001 C CNN
 	1    10550 4600
@@
 BATT_N
 $Comp
-L Switch:SW_SPDT U4
+L solarpcd-rescue:SW_SPDT-Switch U4
 U 1 1 5DCB22FF
 P 10550 5150
 F 0 "U4" H 10550 5435 50  0000 C CNN
 F 1 "SW_SPDT" H 10550 5344 50  0000 C CNN
-F 2 "custom-footprints:D2F-L2" H 10550 5150 50  0001 C CNN
+F 2 "solarpcb:D2F-L2" H 10550 5150 50  0001 C CNN
 F 3 "~" H 10550 5150 50  0001 C CNN
 	1    10550 5150
@@
 	10900 5250 10750 5250
 $Comp
-L Connector:Screw_Terminal_01x02 J3
+L solarpcd-rescue:Screw_Terminal_01x02-Connector J3
 U 1 1 5DCDAA1F
 P 10000 4900
