File: _autosave-ypanel.kicad_pcb (KiCad board)
At the start: 6 copper layers, 64 x 58 mm, 57 parts, among them IC2 TSL2561, J1 XF2M-1015-1A, J2 U.FL-R-SMT-1, J3 BATTERY CONNECTOR, J4 B2B-PH-SM4-TB_LF__SN_, U1 SWLP.12.B, U2 Value, U3 SW_SPDT, U4 SW_SPDT

Commit message: Added step file of -Y
Other:
- outline, holes or cut-outs redrawn
Changed lines of the file:
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@@
   (general
     (thickness 1.6)
-    (drawings 102)
+    (drawings 87)
     (tracks 1713)
     (zones 0)
@@
   )
   (setup
-    (last_trace_width 0.127)
+    (last_trace_width 1)
     (user_trace_width 0.127)
     (user_trace_width 0.16)
@@
     )
   )
-  (gr_circle (center 193 93) (end 195 93) (layer F.SilkS) (width 0.12))
   (gr_line (start 196 110) (end 178 110) (layer F.SilkS) (width 0.12))
   (gr_line (start 196 128) (end 196 110) (layer F.SilkS) (width 0.12))
   (gr_line (start 178 128) (end 196 128) (layer F.SilkS) (width 0.12))
   (gr_line (start 178 110) (end 178 128) (layer F.SilkS) (width 0.12))
-  (gr_circle (center 164.875 118.9) (end 163.775 118.9) (layer Edge.Cuts) (width 0.1))
+  (gr_circle (center 193 93) (end 195 93) (layer F.SilkS) (width 0.12))
   (gr_circle (center 125.075 118.9) (end 127.075 118.9) (layer F.SilkS) (width 0.1))
-  (gr_circle (center 164.875 79.1) (end 163.775 79.1) (layer Edge.Cuts) (width 0.1))
   (gr_circle (center 147.271 99.000001) (end 139.271 99.000001) (layer Edge.Cuts) (width 0.1))
   (gr_circle (center 139.975 113.85) (end 138.945436 113.85) (layer Edge.Cuts) (width 0.1))
   (gr_circle (center 146.45 113.879564) (end 145.420436 113.879564) (layer Edge.Cuts) (width 0.1))
-  (gr_line (start 176.975 128) (end 176.975 70) (layer Edge.Cuts) (width 0.1))
-  (gr_line (start 112.975 128) (end 176.975 128) (layer Edge.Cuts) (width 0.1))
-  (gr_line (start 112.975 128) (end 112.975 70) (layer Edge.Cuts) (width 0.1))
-  (gr_circle (center 164.875 118.9) (end 163.775 118.9) (layer Edge.Cuts) (width 0.1))
-  (gr_line (start 176.975 128) (end 112.975 128) (layer Edge.Cuts) (width 0.1))
   (gr_circle (center 125.075 118.9) (end 126.375 118.9) (layer Edge.Cuts) (width 0.1))
   (gr_circle (center 139.929564 84.15) (end 138.9 84.15) (layer Edge.Cuts) (width 0.1))
-  (gr_circle (center 125.075 79.1) (end 123.975 79.1) (layer Edge.Cuts) (width 0.1))
   (gr_circle (center 146.45 84.15) (end 145.420436 84.15) (layer Edge.Cuts) (width 0.1))
-  (gr_line (start 112.975 70) (end 112.975 128) (layer Edge.Cuts) (width 0.1))
-  (gr_line (start 176.975 70) (end 112.975 70) (layer Edge.Cuts) (width 0.1))
-  (gr_circle (center 125.075 79.1) (end 123.975 79.1) (layer Edge.Cuts) (width 0.1))
-  (gr_circle (center 164.875 79.1) (end 163.775 79.1) (layer Edge.Cuts) (width 0.1))
   (gr_line (start 176.975 70) (end 176.975 128) (layer Edge.Cuts) (width 0.1))
-  (gr_line (start 112.975 70) (end 176.975 70) (layer Edge.Cuts) (width 0.1))
   (gr_text 1 (at 169.1894 83.6676) (layer B.SilkS)
     (effects (font (size 1 1) (thickness 0.1778)) (justify mirror))
@@
   (gr_line (start 113.03 72.9996) (end 177.0172 72.9996) (layer F.SilkS) (width 0.254))
   (gr_line (start 113 125) (end 176.9872 125) (layer F.SilkS) (width 0.254))
-  (gr_circle (center 164.9 118.9) (end 163.8 118.9) (layer Edge.Cuts) (width 0.1))
-  (gr_line (start 177 128) (end 177 70) (layer Edge.Cuts) (width 0.1))
+  (gr_circle (center 164.9 118.9) (end 166.2 118.9) (layer Edge.Cuts) (width 0.1))
   (gr_line (start 168.4 122.4) (end 164.9 122.4) (layer Dwgs.User) (width 0.15))
   (gr_line (start 128.5728 115.3764) (end 121.5728 115.3764) (layer Dwgs.User) (width 0.15))
@@
   (gr_line (start 128.5728 122.3764) (end 128.5728 115.3764) (layer Dwgs.User) (width 0.15))
   (gr_line (start 121.5728 115.3764) (end 121.5728 122.3764) (layer Dwgs.User) (width 0.15))
-  (gr_circle (center 125.0728 118.8764) (end 126.1728 118.8764) (layer Edge.Cuts) (width 0.05))
   (gr_line (start 128.5728 75.6) (end 121.5728 75.6) (layer Dwgs.User) (width 0.15))
   (gr_line (start 121.5728 82.6) (end 128.5728 82.6) (layer Dwgs.User) (width 0.15))
   (gr_line (start 128.5728 82.6) (end 128.5728 75.6) (layer Dwgs.User) (width 0.15))
   (gr_line (start 121.5728 75.6) (end 121.5728 82.6) (layer Dwgs.User) (width 0.15))
-  (gr_circle (center 125.0728 79.1) (end 126.1728 79.1) (layer Edge.Cuts) (width 0.05))
+  (gr_circle (center 125.0728 79.1) (end 126.3728 79.1) (layer Edge.Cuts) (width 0.05))
   (gr_line (start 128.6 75.6) (end 121.6 75.6) (layer Dwgs.User) (width 0.15))
   (gr_line (start 121.6 75.6) (end 121.6 82.6) (layer Dwgs.User) (width 0.15))
@@
   (gr_line (start 168.4 122.4) (end 121.6 122.4) (layer Dwgs.User) (width 0.15))
   (gr_line (start 121.6 75.6) (end 168.4 75.6) (layer Dwgs.User) (width 0.15))
-  (gr_circle (center 164.895 79.10248) (end 163.795 79.10248) (layer Edge.Cuts) (width 0.1))
+  (gr_circle (center 164.895 79.10248) (end 166.195 79.10248) (layer Edge.Cuts) (width 0.1))
   (gr_text coil_p (at 121.031 89.027) (layer B.SilkS)
     (effects (font (size 0.5 0.5) (thickness 0.1)) (justify mirror))
@@
     (effects (font (size 1 1) (thickness 0.15)) (justify mirror))
   )
-  (gr_line (start 177 70) (end 113 70) (layer Edge.Cuts) (width 0.1))
-  (gr_line (start 113 128) (end 177 128) (layer Edge.Cuts) (width 0.1))
+  (gr_line (start 176.975 70) (end 113 70) (layer Edge.Cuts) (width 0.1))
+  (gr_line (start 113 128) (end 176.975 128) (layer Edge.Cuts) (width 0.1))
   (gr_line (start 113 70) (end 113 128) (layer Edge.Cuts) (width 0.1))
   (gr_text v01 (at 141.732 87.1855 180) (layer B.Mask)
@@
   (segment (start 175.713 99.1235) (end 176.32299 98.51351) (width 1) (layer Top) (net 1))
   (segment (start 176.32299 98.51351) (end 176.32299 76.81849) (width 1) (layer Top) (net 1))
-  (segment (start 162.4203 76.2508) (end 162.4203 78.92034) (width 1) (layer Top) (net 1))
-  (segment (start 160.528 74.3585) (end 162.4203 76.2508) (width 1) (layer Top) (net 1))
-  (segment (start 127.277304 74.3585) (end 160.528 74.3585) (width 1) (layer Top) (net 1))
-  (segment (start 121.92 79.715804) (end 127.277304 74.3585) (width 1) (layer Top) (net 1))
-  (segment (start 121.92 95.758) (end 121.92 79.715804) (width 1) (layer Top) (net 1))
   (segment (start 130.85 100.65) (end 130.85 102.65) (width 1) (layer Top) (net 1))
   (segment (start 126.2 96) (end 130.85 100.65) (width 1) (layer Top) (net 1))
@@
   (segment (start 163.09848 82.8) (end 162.4203 82.12182) (width 1) (layer Top) (net 1))
   (segment (start 163.09848 84.8) (end 163.09848 82.8) (width 1) (layer Top) (net 1))
+  (segment (start 162.4203 76.2508) (end 162.4203 78.92034) (width 1) (layer Top) (net 1))
+  (segment (start 160.528 74.3585) (end 162.4203 76.2508) (width 1) (layer Top) (net 1))
+  (segment (start 127.025683 74.3585) (end 160.528 74.3585) (width 1) (layer Top) (net 1))
+  (segment (start 121.92 79.464183) (end 127.025683 74.3585) (width 1) (layer Top) (net 1))
+  (segment (start 121.92 95.758) (end 121.92 79.464183) (width 1) (layer Top) (net 1))
   (via (at 150.19782 86.07298) (size 0.6) (drill 0.3) (layers Top Bottom) (net 2))
   (via (at 144.9324 78.8416) (size 0.6) (drill 0.3) (layers Top Bottom) (net 2))
