File: ypanel.kicad_pcb (KiCad board)
At the start: 6 copper layers, 64 x 58 mm, 61 parts, among them IC2 TSL2561, J1 XF2M-1015-1A, J2 Conn_Coaxial, J3 BATTERY CONNECTOR, J4 B2B-PH-SM4-TB_LF__SN_, U2 Value, U3 SW_SPDT, U4 SW_SPDT

Commit message: fixing coil-to-board-edge distance...
Routing:
- net /coil: track 16804.8 -> 16779.6 mm

Commit message: -y panel coils fixed and manufacturing files generated
Routing:
- net /coil: track 16779.6 -> 16749.1 mm
